File: hw/cube.kicad_sch (KiCad schematic)
At the start: 63 parts, among them J1 USB-C, J2 ECRAN QSPI, J3 microSD, J4 HP, J5 I2C EXT, J6 DEBUG, SW1 RESET, SW2 BOOT, U1 AP63203WU, U2 ESP32-S3-WROOM-1U-N16R8, U3 MAX98357A, U4 VL53L1X, U5 LIS3DH

Commit message: feat(hw): carte entierement routee — 223/223 connexions
Les 4 dernieres liaisons, autour du LIS3DH (LGA-16 au pas de 0,5 mm), ont ete
tirees a la main dans Pcbnew. La masse de U5 passe par une piste sur In2.Cu et
un via vers le plan : cela cree une fente courte dans le plan +3V3, dans un
coin qui ne consomme que des microamperes, donc sans consequence.

tools/import_routes.py recapture ce cuivre dans routes.json : le routage
manuel fait desormais partie du pipeline au lieu d'etre perdu a la prochaine
generation. Le format accepte un nom de couche et la taille reelle des vias,
ce qu'exigeaient la piste sur couche interne et les vias 0,7/0,35.

Corrections associees, toutes signalees par le DRC :
- serigraphie remontee de 0,6 a 0,8 mm : sous 0,8 mm le texte n'est pas
  garanti lisible par le fabricant (75 avertissements) ;
- H1-H4 et TP1-TP4 declares hors nomenclature cote schema, les empreintes
  portaient deja le drapeau (8 divergences empreinte/symbole) ;
- deux moignons de 0,1 mm sur USB_DM supprimes.

Etat : 0 erreur ERC, 0 violation DRC, 0 liaison non routee, 0 ecart de parite.
Restent 8 avertissements de serigraphie cosmetiques.
Parts:
- H1, H2, H3, H4, TP1, TP2, TP3, TP4: now left out of the parts list
Changed lines of the file:
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@@
 	(title_block
 		(title "CUBE - Afficheur holographique Pepper's Ghost")
-		(date "2026-08-24")
+		(date "2026-08-27")
 		(rev "A")
 		(comment 1 "ESP32-S3-WROOM-1U-N16R8 / AMOLED QSPI / microSD SDIO")
@@
 		(unit 1)
 		(exclude_from_sim no)
-		(in_bom yes)
+		(in_bom no)
 		(on_board yes)
 		(dnp no)
@@
 		(unit 1)
 		(exclude_from_sim no)
-		(in_bom yes)
+		(in_bom no)
 		(on_board yes)
 		(dnp no)
@@
 		(unit 1)
 		(exclude_from_sim no)
-		(in_bom yes)
+		(in_bom no)
 		(on_board yes)
 		(dnp no)
@@
 		(unit 1)
 		(exclude_from_sim no)
-		(in_bom yes)
+		(in_bom no)
 		(on_board yes)
 		(dnp no)
@@
 		(unit 1)
 		(exclude_from_sim no)
-		(in_bom yes)
+		(in_bom no)
 		(on_board yes)
 		(dnp no)
@@
 		(unit 1)
 		(exclude_from_sim no)
-		(in_bom yes)
+		(in_bom no)
 		(on_board yes)
 		(dnp no)
@@
 		(unit 1)
 		(exclude_from_sim no)
-		(in_bom yes)
+		(in_bom no)
 		(on_board yes)
 		(dnp no)
@@
 		(unit 1)
 		(exclude_from_sim no)
-		(in_bom yes)
+		(in_bom no)
 		(on_board yes)
 		(dnp no)
